Commit message: update tf2
update moveable frame of robot

File: franka_description/robots/panda_arm_rbdl_origin_copy_.urdf (robot description, URDF)
Before this commit: robot panda, 12 links, 11 joints
Links:
- removed link panda_link_target
- added link panda_rightfinger; visual mesh filename=package://franka_description/meshes/visual/finger.dae
- link panda_link0: mass 1.43675504024173 -> None; geometry collision cylinder length=0.03 radius=0.09; collision sphere radius=0.09
- link panda_link1: mass 1.43675504024173 -> None; geometry collision cylinder length=0.2830 radius=0.09; collision sphere radius=0.09
- link panda_link2: mass 1.43675504024173 -> None; geometry collision cylinder length=0.12 radius=0.09; collision sphere radius=0.09
- link panda_link3: mass 1.43675504024173 -> None; geometry collision cylinder length=0.15 radius=0.09; collision sphere radius=0.09
- link panda_link4: mass 1.43675504024173 -> None; geometry collision cylinder length=0.12 radius=0.09; collision sphere radius=0.09
- link panda_link5: mass 1.43675504024173 -> None; geometry collision cylinder length=0.1 radius=0.09; collision cylinder length=0.14 radius=0.055
- link panda_link6: mass 1.43675504024173 -> None; geometry collision cylinder length=0.08 radius=0.08; collision sphere radius=0.08
- link panda_link7: mass 1.43675504024173 -> None; geometry collision cylinder length=0.14 radius=0.07; collision sphere radius=0.07
Joints:
- removed joint panda_link_target
- added joint panda_finger_joint2: type prismatic, parent panda_hand, child panda_rightfinger, origin xyz=0 0 0.0584 rpy=0 0 0, axis 0 -1 0, limit lower=0.0 upper=0.04 effort=20 velocity=0.2, mimic joint=panda_finger_joint1
